File: EmuBoard2350/EmuBoard2350.kicad_pcb (KiCad board)
At the start: 4 copper layers, 87 x 71 mm, 109 parts, among them J1 USB_C_Receptacle_USB2.0_16P, J10 KF141V, J11 USB_A, J12 Conn_01x10, J13 Conn_01x04, J2 Barrel_Jack_Switch, J3 Conn_01x03, J4 HDMI_A, J5 Mini-DIN-6, J6 Mini-DIN-6, J7 Micro_SD_Card, J8 PJ-307, J9 Conn_01x10, Q1 2N7002, Q2 2N7002, Q3 2N7002, Q4 2N7002, SW1 SW_Push, SW2 SW_Push, U1 RP2350B, U2 W25Q128JVS, U3 AMS1117-3.3, U4 KA78M05_TO252, U5 APS6404L_3SQRSN, U6 PCM5102A, Y1 12 MHz

Commit message: JLCPCB Order
Parts:
- added C18: 10 uF, Capacitor_SMD:C_0603_1608Metric, F.Cu at (153.5, 104.5)
- added C38: 100 nF, Capacitor_SMD:C_0402_1005Metric, F.Cu at (141.7, 71.7)
- added C39: 100 nF, Capacitor_SMD:C_0402_1005Metric, F.Cu at (139.8, 73.5)
- J13: value Conn_01x04 -> Conn_01x06; footprint EmuBoard2350:KF141-terminal-block-4pos -> EmuBoard2350:KF141-terminal-block-6pos
- L1: footprint EmuBoard2350:abracon_aota-b201610s3r3-101-t -> Inductor_SMD:L_1008_2520Metric
- moved R26 6.32 mm to (159.3, 106.9)
- moved R1 4.39 mm to (147.4, 93.3), turned to -90 degrees
- moved R24 4.39 mm to (162.5, 106.9)
- moved R25 4.37 mm to (156.8, 106.3), turned to 90 degrees
- moved R28 4.35 mm to (166.6, 106.8)
- moved J8 3.10 mm to (161.7, 115.9)
- moved R6 2.80 mm to (139.9, 68.6)
- moved R5 2.58 mm to (141.8, 68.9)
- moved R37 1.91 mm to (150.0, 104.5)
- moved C27 0.78 mm to (137.5, 92.0)
- moved J13 0.73 mm to (161.2, 87.5)
- moved L1 0.51 mm to (142.4, 73.7)
- moved C11 0.47 mm to (139.4, 92.0)
- moved C22 0.31 mm to (136.2, 91.4)
Connections:
- J13 pad 1: +3.3V -> /GPIO30
- J13 pad 2: Net-(J13-Pin_2) -> /GPIO29
- J13 pad 3: /GPIO30 -> /GPIO28
- J13 pad 4: GND -> Net-(J13-Pin_4)
- R37 pad 1: Net-(J13-Pin_2) -> Net-(J13-Pin_4)
- U1 pad 36: unconnected-(U1-GPIO28-Pad36) -> /GPIO28
- U1 pad 37: unconnected-(U1-GPIO29-Pad37) -> /GPIO29
Routing:
- net Net-(J13-Pin_4): track 0.00 -> 52.2 mm, vias 0 -> 1
- net Net-(J13-Pin_2): track 46.3 -> 0.00 mm, vias 1 -> 0
- net /GPIO28: track 0.00 -> 34.1 mm, vias 0 -> 1
- net /GPIO29: track 0.00 -> 31.3 mm, vias 0 -> 1
- net Net-(J10-Pin_5): track 17.8 -> 26.6 mm
- net Net-(J10-Pin_6): track 19.0 -> 26.8 mm
- net /GPIO30: track 35.2 -> 29.2 mm
- net +3.3V: track 92.8 -> 87.1 mm, vias 44 -> 43
- net /NESDATA1: track 37.4 -> 42.5 mm
- net Net-(J11-D-): track 36.9 -> 32.2 mm
- net Net-(C35-Pad2): track 15.8 -> 20.4 mm
- net /NESDATA2: track 43.1 -> 47.5 mm
- net +1V1: track 47.1 -> 51.3 mm
- net Net-(J11-D+): track 36.8 -> 33.2 mm
- net GND: track 176.5 -> 173.0 mm, vias 81 -> 84
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Other:
- board text added: "28"
- board text added: "29"
- board text added: "POWER 7.5-9 VDC CENTER POS"
- board text removed: "POWER 7-12 VDC CENTER POS"
