File: EmuBoard2350/EmuBoard2350.kicad_sch (KiCad schematic)
At the start: 109 parts, among them J1 USB_C_Receptacle_USB2.0_16P, J10 KF141V, J11 USB_A, J12 Conn_01x10, J13 Conn_01x04, J2 Barrel_Jack_Switch, J3 Conn_01x03, J4 HDMI_A, J5 Mini-DIN-6, J6 Mini-DIN-6, J7 Micro_SD_Card, J8 PJ-307, J9 Conn_01x10, Q1 2N7002, Q2 2N7002, Q3 2N7002, Q4 2N7002, SW1 SW_Push, SW2 SW_Push, U1 RP2350B, U2 W25Q128JVS, U3 AMS1117-3.3, U4 KA78M05_TO252, U5 APS6404L_3SQRSN, U6 PCM5102A, Y1 12 MHz

Commit message: JLCPCB Order
Parts:
- removed J13: Conn_01x04, EmuBoard2350:KF141-terminal-block-4pos, symbol Connector_Generic:Conn_01x04
- added C18: 10 uF, Capacitor_SMD:C_0603_1608Metric, symbol Device:C_Small
- added C38, C39: 100 nF, Capacitor_SMD:C_0402_1005Metric, symbol Device:C_Small
- added J13: Conn_01x06, EmuBoard2350:KF141-terminal-block-6pos, symbol Connector_Generic:Conn_01x06
- C1: LCSC (none) -> DNP; now not fitted
- C12, C14, C15, C7: LCSC C1705 -> C19666
- C16, C17, C30, C33, C34: LCSC C1691 -> C19702
- H1, H2, H3, H4, J10, J12, J2, J3, J5, J6, J9: now not fitted
- J1: FT Position Offset (none) -> 0.0,2.54
- J4: FT Rotation Offset (none) -> 90
- J7: FT Rotation Offset (none) -> 180
- J8: FT Position Offset (none) -> 0,-2.54
- L1: footprint EmuBoard2350:abracon_aota-b201610s3r3-101-t -> Inductor_SMD:L_1008_2520Metric; LCSC C42411119 -> C5832359
- R1, R2, R23, R29, R30, R31, R32, R33, R34, R35, R40, R41, R42: LCSC C174175 -> C25744
- U1: FT Rotation Offset (none) -> -90; LCSC C42415655 -> (none); private KLC_S4.2_DVDD -> (none)
- Y1: LCSC C9002 -> C20625731
Connections:
- net +1V1: now also C38.1, C39.1
- net +3.3V: now also J13.5 (Pin_5)
- net GND: now also C18.2, C38.2, C39.2, J13.6 (Pin_6)
- net GPIO30: now also J13.1 (Pin_1)
- net at R37.1: now also C18.1, J13.4 (Pin_4)
- net GPIO28: now reaches U1.36 (GPIO28)
- net GPIO28: now also J13.3 (Pin_3)
- net GPIO29: now reaches U1.37 (GPIO29)
- net GPIO29: now also J13.2 (Pin_2)
